Commit message: add a tcp link to urdf

File: urdf/arm.urdf (robot description, URDF)
Before this commit: robot arm.SLDASM, 7 links, 6 joints
Links:
- added link Link_tcp
Joints:
- added joint Joint_tcp: type fixed, parent Link_3, child Link_tcp, origin xyz=0.14565 0 -0.02045 rpy=0 0 0

Commit message: add target ee control

File: urdf/arm.urdf (robot description, URDF)
Before this commit: robot arm.SLDASM, 8 links, 7 joints
Joints:
- joint Joint_0: axis 0 0 -1 -> 0 0 1
- joint Joint_1: axis 0 -1 0 -> 0 1 0
- joint Joint_2: axis 0 -1 0 -> 0 1 0; limit lower=-0.75 upper=1.77 effort=0 velocity=0 -> lower=-1.77 upper=0.75 effort=0 velocity=0
- joint Joint_3: axis 0 -1 0 -> 0 1 0

File: urdf/robot.urdf (robot description, URDF)
Before this commit: robot create3, 14 links, 13 joints
Joints:
- joint Joint_0: axis 0 0 -1 -> 0 0 1
- joint Joint_1: axis 0 -1 0 -> 0 1 0
- joint Joint_2: axis 0 -1 0 -> 0 1 0; limit lower=-0.75 upper=1.77 effort=0 velocity=0 -> lower=-1.77 upper=0.75 effort=0 velocity=0
- joint Joint_3: axis 0 -1 0 -> 0 1 0
