Commit message: add mobile base's control to simulation envs

File: urdf/robot.urdf (robot description, URDF)
Before this commit: robot create3, 10 links, 9 joints
Links:
- added link theta_link
- added link world_link
- added link x_link
- added link y_link
Joints:
- added joint base_joint: type fixed, parent theta_link, child base_link, origin xyz=0 0 0
- added joint theta_joint: type revolute, parent y_link, child theta_link, origin xyz=0 0 0, axis 0 0 1, limit lower=-6.28 upper=6.28 effort=0 velocity=0
- added joint x_joint: type prismatic, parent world_link, child x_link, origin xyz=0 0 0, axis 1 0 0, limit lower=-5 upper=5 effort=0 velocity=0
- added joint y_joint: type prismatic, parent x_link, child y_link, origin xyz=0 0 0, axis 0 1 0, limit lower=-5 upper=5 effort=0 velocity=0

Commit message: transfer from gym to gymnasium

File: urdf/robot.urdf (robot description, URDF)
Before this commit: robot create3, 14 links, 13 joints
Joints:
- joint Joint_1: limit lower=-1.63 upper=1.63 effort=0 velocity=0 -> lower=-1.0 upper=1.0 effort=0 velocity=0
- joint Joint_2: limit lower=-1.77 upper=0.75 effort=0 velocity=0 -> lower=-1.0 upper=0.7 effort=0 velocity=0
- joint Joint_3: limit lower=-1.77 upper=1.77 effort=0 velocity=0 -> lower=-1.1 upper=1.1 effort=0 velocity=0
